File: hardware/wfoc/wfoc.kicad_sch (KiCad schematic)
At the start: 72 parts, among them Q1 NMOS, Q2 NMOS, Q3 NMOS, Q4 NMOS, Q5 NMOS, Q6 NMOS, U3 TSSOP20

Commit message: 修改PCB板连线
Parts:
- removed C1, C2: 101, symbol Device:C
- removed R13, R14: 100R, symbol Device:R
- added R4, R6: 0.0025R 1%, Resistor_SMD:R_2512_6332Metric, symbol Device:R
- C10, C14, C15, C16, C17, C18, C3, C4, C5, C6, C7, C8: footprint (none) -> Capacitor_SMD:C_0603_1608Metric
- C11, C9: footprint (none) -> Capacitor_THT:CP_Radial_D10.0mm_P7.50mm
- C12, C13: footprint (none) -> Capacitor_SMD:C_0805_2012Metric
- D1: footprint (none) -> Diode_SMD:D_1206_3216Metric_Pad1.42x1.75mm_HandSolder
- EG1192L1: footprint ESOP8 -> Package_SO:SOP-8-1EP_6.0x4.9mm_P1.27mm_EP2.4x3.3mm
- L1: value 47uH -> 47uH GSM0650-470-M; footprint (none) -> Inductor_SMD:L_7.5x6.6mm
- Q1, Q2, Q3, Q4, Q5, Q6: footprint (none) -> Package_TO_SOT_SMD:TO-252-2
- R1, R2: value 0.005R 1% -> 0.0025R 1%; footprint (none) -> Resistor_SMD:R_2512_6332Metric
- R10, R11, R12, R15, R16, R17, R19, R20, R21, R22, R23, R24, R25, R26, R27, R28, R29, R3, R30, R31, R32, R33, R35, R36, R37, R38, R5, R7, R8, R9, TH1: footprint (none) -> Resistor_SMD:R_0603_1608Metric
- R18: footprint (none) -> Resistor_SMD:R_1206_3216Metric
- R40: renamed from 47K; footprint (none) -> Resistor_SMD:R_0603_1608Metric
- R41: renamed from R31; value 10K -> 47K; footprint (none) -> Resistor_SMD:R_0603_1608Metric
- R42: renamed from R32; footprint (none) -> Resistor_SMD:R_0603_1608Metric
- R43: renamed from R33; value 10K -> 47K; footprint (none) -> Resistor_SMD:R_0603_1608Metric
- R44: renamed from 10K; footprint (none) -> Resistor_SMD:R_0603_1608Metric
- U1: footprint (none) -> Package_DFN_QFN:QFN-20-1EP_3x3mm_P0.4mm_EP1.5x1.5mm
- U2: footprint (none) -> Package_SO:SOP-8_3.9x4.9mm_P1.27mm
- U3: footprint (none) -> Package_SO:TSSOP-20_4.4x6.5mm_P0.65mm
- U4: value (none) -> 6209; footprint (none) -> Package_TO_SOT_SMD:SOT-23
Connections:
- net +3.3V: now also U4.2 (VOut); no longer U4. (VOut)
- net +BATT: now also EG1192L1.9 (VIN), Q1.2 (D), Q2.2 (D), Q3.2 (D); no longer EG1192L1.0 (VIN), Q1.1 (D), Q2.1 (D), Q3.1 (D)
- net GNDMotor: now also C10.1, C11.2, C12.1, C13.1, C14.1, C15.2, C5.2, C8.1, C9.2, D1.2 (A), EG1192L1.2 (GND), Q5.3 (S), R11.2, R15.2, R20.2, R31.2, R35.1, R36.1, R37.1, R38.1, TH1.2, U1.4 (VSS), U2.4 (-VS), U3.8 (COM), U4.1 (GND), R4.1, R6.1
- net IC_ia: now also R9.1, U2.7 (OUTB)
- net IC_ib: now also R7.1, U2.1 (OutA)
- net Ia_P: now also R6.2
- net Ib_P: now also R4.2
- net LO1: now also Q4.1 (G); no longer Q4.2 (G)
- net LO2: now also Q6.1 (G); no longer Q6.2 (G)
- net LO3: now also Q5.1 (G); no longer Q5.2 (G)
- net Motor_U: now also Q4.2 (D); no longer Q4.1 (D)
- net Motor_V: now also Q6.2 (D); no longer Q6.1 (D)
- net Motor_W: now also Q5.2 (D); no longer Q5.1 (D)
- net at R23.2, R29.1: now also Q2.1 (G); no longer Q2.2 (G)
- net at R22.2, R30.1: now also Q3.1 (G); no longer Q3.2 (G)
- net at C13.2, R21.1: now also U4.3 (Vin); no longer U4. (VOut)
- net at R24.2, R28.1: now also Q1.1 (G); no longer Q1.2 (G)
- removed net GNDREF: C10.1, C11.2, C12.1, C13.1, C14.1, C15.2, C5.2, C8.1, C9.2, D1.2 (A), EG1192L1.2 (GND), Q5.3 (S), R11.2, R15.2, R20.2, R31.2, R35.1, R36.1, R37.1, R38.1, TH1.2, U1.4 (VSS), U2.4 (-VS), U3.8 (COM), U4. (VOut)

Commit message: 提交最新的readme 和hardware改动
Parts:
- added C19, C20: 103, Capacitor_SMD:C_0603_1608Metric, symbol Device:C
- added R13, R14: 100R, Resistor_SMD:R_0603_1608Metric, symbol Device:R
- R40: value 10K -> 39K
- R41, R42, R43: value 47K -> 39K
- TH1: value 10K NTC 4390K -> 10K NTC 3490K
- U2: value (none) -> XOPA2333
Connections:
- net +3.3V: now also TH1.2; no longer R44.2
- net GNDMotor: now also R44.2, C19.1, C20.1; no longer TH1.2
- net IC_ia: now also C19.2, R14.2; no longer R9.1, U2.7 (OUTB)
- net IC_ib: now also C20.2, R13.1; no longer R7.1, U2.1 (OutA)
- new net: R13.2, R7.1, U2.1 (OutA)
- new net: R14.1, R9.1, U2.7 (OUTB)
Other:
- moved on the sheet: R44, TH1
