File: hardware/wfoc/wfoc.kicad_sch (KiCad schematic)
At the start: 70 parts, among them Q1 NMOS, Q2 NMOS, Q3 NMOS, Q4 NMOS, Q5 NMOS, Q6 NMOS, U3 TSSOP20, U4 6209

Commit message: save last vesion
Parts:
- R40: value 10K -> 47K; footprint Resistor_SMD:R_0603_1608Metric -> Resistor_SMD:R_0805_2012Metric
Changed lines of the file:
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@@
 			)
 		)
-		(property "Value" "10K"
+		(property "Value" "47K"
 			(at 130.048 82.804 0)
 			(show_name no)
@@
 			)
 		)
-		(property "Footprint" "Resistor_SMD:R_0603_1608Metric"
+		(property "Footprint" "Resistor_SMD:R_0805_2012Metric"
 			(at 128.778 86.36 90)
 			(hide yes)

Commit message: 基本画好 还有些信号线没有连上了
Parts:
- added C19, C20: 103, Capacitor_SMD:C_0603_1608Metric, symbol Device:C
- added R13, R14: 100R, Resistor_SMD:R_0603_1608Metric, symbol Device:R
- R1, R2, R4, R6: value 0.0025R 1% -> 0.005R 1%
- R22, R23, R24, R25, R26, R27: value 22R -> 10R
- R36, R37, R38, R44: footprint Resistor_SMD:R_0603_1608Metric -> Resistor_SMD:R_0402_1005Metric
- U2: value (none) -> XOPA2333
Connections:
- net +3.3V: now also TH1.2; no longer R44.2
- net GNDMotor: now also R44.2, C19.1, C20.2; no longer TH1.2
- net IC_ia: now also C20.1, R14.2; no longer R9.1, U2.7 (OUTB)
- net IC_ib: now also C19.2, R13.1; no longer R7.1, U2.1 (OutA)
- new net: R14.1, R9.1, U2.7 (OUTB)
- new net: R13.2, R7.1, U2.1 (OutA)
Other:
- moved on the sheet: R44, TH1
