File: hardware/wfoc/wfoc.kicad_pcb (KiCad board)
At the start: 2 copper layers, 50 x 50 mm, 70 parts, among them Q1 NMOS, Q2 NMOS, Q3 NMOS, Q4 NMOS, Q5 NMOS, Q6 NMOS, U3 TSSOP20, U4 6209

Commit message: save last vesion
Parts:
- R25, R26, R27, R31, R32, R33: moved to F.Cu
- R40: value 10K -> 47K; footprint Resistor_SMD:R_0603_1608Metric -> Resistor_SMD:R_0805_2012Metric
- moved C14 37.2 mm to (154.7, 95.0), turned to 180 degrees
- moved R44 29.2 mm to (120.5, 103.7), turned to 90 degrees
- moved U3 29.1 mm to (152.6, 90.4), turned to 90 degrees
- moved C18 24.6 mm to (155.8, 85.0), turned to 180 degrees
- moved C17 23.0 mm to (152.7, 85.5), turned to 180 degrees
- moved C16 21.7 mm to (150.2, 85.0), turned to -90 degrees
- moved R20 6.84 mm to (153.5, 106.0), turned to 90 degrees
- moved R10 6.52 mm to (130.1, 90.0)
- moved R12 6.52 mm to (121.1, 91.5)
- moved R16 6.52 mm to (121.1, 88.2)
- moved R2 6.52 mm to (138.6, 88.6)
- moved R3 6.52 mm to (130.1, 87.0)
- moved R4 6.52 mm to (143.1, 88.5)
- moved R5 6.52 mm to (130.1, 88.5)
- moved R8 6.52 mm to (130.1, 91.5)
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Routing:
- net +BATT: track 0.00 -> 55.3 mm
- net PWM_AH: track 0.00 -> 28.7 mm
- net +12V: track 0.00 -> 18.3 mm
- net Net-(U3-LO2): track 29.8 -> 13.3 mm
- net PWM_CL: track 0.00 -> 13.8 mm
- net Net-(D1-K): track 0.00 -> 13.2 mm
- net PWM_BL: track 0.00 -> 13.0 mm
- net Net-(U3-LO1): track 4.26 -> 16.9 mm
- net Net-(U3-HO1): track 4.45 -> 15.0 mm
- net Net-(U3-HO2): track 3.18 -> 11.9 mm
- net PWM_AL: track 0.00 -> 8.58 mm
- net Net-(U3-LO3): track 17.6 -> 9.53 mm
- net PWM_CH: track 0.00 -> 7.12 mm
- net Ia_P: track 19.0 -> 12.3 mm, vias 0 -> 1
- net LO3: track 0.00 -> 6.47 mm, vias 0 -> 1
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
Commit message: 基本画好 还有些信号线没有连上了
Parts:
- added C19: 103, Capacitor_SMD:C_0603_1608Metric, F.Cu at (121.7, 98.0)
- added C20: 103, Capacitor_SMD:C_0603_1608Metric, F.Cu at (123.7, 100.5)
- added R13: 100R, Resistor_SMD:R_0603_1608Metric, F.Cu at (121.8, 96.5)
- added R14: 100R, Resistor_SMD:R_0603_1608Metric, F.Cu at (124.8, 99.0)
- R1, R2, R4, R6: value 0.0025R 1% -> 0.005R 1%
- R22, R23, R24, R25, R26, R27: value 22R -> 10R
- R36, R37, R38, R44: footprint Resistor_SMD:R_0603_1608Metric -> Resistor_SMD:R_0402_1005Metric
- U2: value ~ -> XOPA2333
- moved R38 33.9 mm to (120.0, 101.5), turned to 180 degrees
- moved R36 8.06 mm to (119.0, 104.0), turned to 180 degrees
- moved R35 7.56 mm to (123.2, 106.5), turned to 0 degrees
- moved R37 5.99 mm to (119.5, 103.0)
- moved TH1 5.41 mm to (124.0, 72.8), turned to 90 degrees
- moved R44 2.82 mm to (123.0, 105.0), turned to 180 degrees
- moved C5 2.28 mm to (130.5, 104.0), turned to -90 degrees
- moved R41 1.71 mm to (130.2, 68.5)
- moved C4 1.48 mm to (124.8, 96.5)
- moved C10 1.00 mm to (150.0, 99.7)
- moved U1 0.90 mm to (126.5, 104.1), turned to 90 degrees
- moved R21 0.87 mm to (141.8, 100.5)
- moved C15 0.82 mm to (147.3, 99.2), turned to 90 degrees
- moved R42 0.61 mm to (142.7, 68.0), turned to 0 degrees
- moved C13 0.50 mm to (139.0, 99.5)
Connections:
- R44 pad 2: +3.3V -> Ia_N
- R7 pad 1: IC_ib -> Net-(U2-OutA)
- R9 pad 1: IC_ia -> Net-(U2-OUTB)
- TH1 pad 2: Ia_N -> +3.3V
- U2 pad 1: IC_ib -> Net-(U2-OutA)
- U2 pad 7: IC_ia -> Net-(U2-OUTB)
Routing:
- net Vol_W: track 0.00 -> 73.9 mm
- net Vol_V: track 0.00 -> 63.2 mm
- net Vol_U: track 0.00 -> 51.9 mm
- net PWM_BH: track 5.76 -> 39.5 mm, vias 0 -> 2
- net PWM_BL: track 13.0 -> 38.9 mm, vias 0 -> 2
- net PWM_CH: track 7.12 -> 30.6 mm
- net PWM_AL: track 8.58 -> 29.7 mm, vias 0 -> 2
- net +12V: track 18.3 -> 37.0 mm
- net +3.3V: track 9.43 -> 28.2 mm, vias 0 -> 1
- net PWM_CL: track 13.8 -> 31.8 mm
- net Net-(U2-OUTB): track 0.00 -> 17.8 mm
- net SWCLK: track 0.00 -> 9.53 mm, vias 0 -> 1
- net IC_ib: track 2.12 -> 9.99 mm, vias 0 -> 2
- net UartTX: track 0.00 -> 6.67 mm, vias 0 -> 1
- net SWDIO: track 0.00 -> 6.63 mm, vias 0 -> 3
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