File: hardware/wfoc/_restore_backup_2026-07-17T01-08-03-679/wfoc.kicad_sch (KiCad schematic)
At the start: 77 parts, among them Q1 NMOS, Q2 NMOS, Q3 NMOS, Q4 NMOS, Q5 NMOS, Q6 NMOS, U2 XOPA2333, U3 TSSOP20, U4 6209

Commit message: 提交最后板子修改版本
Parts:
- added R39: 2K, Resistor_SMD:R_0402_1005Metric, symbol Device:R
- R45, R46, R47: footprint Resistor_SMD:R_0402_1005Metric -> Resistor_SMD:R_0603_1608Metric
Connections:
- net GNDMotor: now also U1.21 (GND)
- net Vol_U: no longer R45.1
- net Vol_V: no longer R46.1
- net Vol_W: no longer R47.1
- new net CLK: R46.1
- new net CSN: R45.1
- new net Hall_C: R39.2, R47.1
- new net MISO: R39.1
